File: VhfAmTxDrive/VhfAmTxDrive.kicad_pcb (KiCad board)
At the start: 2 copper layers, 45 x 46 mm, 22 parts, among them J1 SMA_EdgeMount, J2 Conn_01x02, J3 SMA_EdgeMount, Q1 2SC4703

Commit message: 基板修正
Parts:
- moved R4 2.25 mm to (75.8, 59.7)
- moved C4 1.53 mm to (77.5, 59.7)
Connections:
- Q1 pad 2: Net-(Q1-E) -> Net-(Q1-C)
- Q1 pad 3: Net-(Q1-C) -> Net-(Q1-E)
Routing:
- net Net-(Q1-C): track 20.5 -> 27.7 mm
- net GND: vias 92 -> 90
Other:
- board text added: "VHF AM TX Driver v0.3"
- board text removed: "VHF AM TX Driver v0.2"
Changed lines of the file:
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@@
 	(footprint "Capacitor_SMD:C_0603_1608Metric_Pad1.08x0.95mm_HandSolder"
 		(layer "F.Cu")
-		(at 75.975 59.6625 90)
+		(at 77.5 59.6625 90)
 		(descr "Capacitor SMD 0603 (1608 Metric), square (rectangular) end terminal, IPC-7351 nominal with elongated pad for handsoldering. (Body size source: IPC-SM-782 page 76, https://www.pcb-3d.com/wordpress/wp-content/uploads/ipc-sm-782a_amendment_1_and_2.pdf), generated with kicad-footprint-generator")
 		(tags "capacitor handsolder")
 		(property "Reference" "C4"
-			(at -2.3375 -0.375 180)
+			(at -2.3375 0.25 180)
 			(layer "F.SilkS")
 			(effects
@@
 		(tags "SOT-89-3 Handsoldering")
 		(property "Reference" "Q1"
-			(at 4.075 0 180)
+			(at 4.975 0 180)
 			(layer "F.SilkS")
 			(effects
@@
 			)
 		)
-		(property "Description" "NPN transistor, base/emitter/collector"
+		(property "Description" "NPN transistor, base/collector/emitter"
 			(at 0 0 90)
 			(unlocked yes)
@@
 			(size 2.475 0.9)
 			(layers "F.Cu" "F.Mask" "F.Paste")
-			(net 5 "Net-(Q1-E)")
-			(pinfunction "E")
+			(net 6 "Net-(Q1-C)")
+			(pinfunction "C")
 			(pintype "passive")
 			(zone_connect 2)
@@
 			(layers "F.Cu" "F.Mask" "F.Paste")
 			(roundrect_rratio 0.25)
-			(net 6 "Net-(Q1-C)")
-			(pinfunction "C")
+			(net 5 "Net-(Q1-E)")
+			(pinfunction "E")
 			(pintype "passive")
 		)
@@
 	(footprint "Resistor_SMD:R_0603_1608Metric_Pad0.98x0.95mm_HandSolder"
 		(layer "F.Cu")
-		(at 78 59.7125 -90)
+		(at 75.75 59.6625 -90)
 		(descr "Resistor SMD 0603 (1608 Metric), square (rectangular) end terminal, IPC-7351 nominal with elongated pad for handsoldering. (Body size source: IPC-SM-782 page 72, https://www.pcb-3d.com/wordpress/wp-content/uploads/ipc-sm-782a_amendment_1_and_2.pdf), generated with kicad-footprint-generator")
 		(tags "resistor handsolder")
 		(property "Reference" "R4"
-			(at 2.2875 -0.2 180)
+			(at 2.2875 0.25 180)
 			(layer "F.SilkS")
 			(effects
@@
 		(layer "Edge.Cuts")
 	)
-	(gr_text "VHF AM TX Driver v0.2"
+	(gr_text "VHF AM TX Driver v0.3"
 		(at 91 39 0)
 		(layer "B.SilkS")
@@
 	)
 	(via
+		(at 80.25 52.5)
+		(size 0.6)
+		(drill 0.3)
+		(layers "F.Cu" "B.Cu")
+		(free yes)
+		(net 2)
+	)
+	(via
 		(at 63 68.2)
 		(size 0.6)
@@
 	)
 	(via
+		(at 77.75 51.5)
+		(size 0.6)
+		(drill 0.3)
+		(layers "F.Cu" "B.Cu")
+		(free yes)
+		(net 2)
+	)
+	(via
 		(at 81.6 42.2)
 		(size 0.6)
@@
 	)
 	(via
+		(at 77.75 50.5)
+		(size 0.6)
+		(drill 0.3)
+		(layers "F.Cu" "B.Cu")
+		(free yes)
+		(net 2)
+	)
+	(via
 		(at 56 48.6)
 		(size 0.6)
@@
 	)
 	(via
+		(at 75.25 49.5)
+		(size 0.6)
+		(drill 0.3)
+		(layers "F.Cu" "B.Cu")
+		(free yes)
+		(net 2)
+	)
+	(via
 		(at 92.6 52.6)
 		(size 0.6)
@@
 	)
 	(via
-		(at 81.6 51.8)
+		(at 81.5 51.75)
 		(size 0.6)
 		(drill 0.3)
@@
 	)
 	(via
-		(at 78.4 54.6)
-		(size 0.6)
-		(drill 0.3)
-		(layers "F.Cu" "B.Cu")
-		(free yes)
-		(net 2)
-	)
-	(via
 		(at 56 71.8)
 		(size 0.6)
@@
 	)
 	(via
-		(at 77 60)
+		(at 76.75 60.5)
 		(size 0.6)
 		(drill 0.3)
@@
 	)
 	(via
-		(at 99 72.2)
+		(at 78.75 55.75)
 		(size 0.6)
 		(drill 0.3)
@@
 	)
 	(via
-		(at 59.8 46.6)
+		(at 99 72.2)
 		(size 0.6)
 		(drill 0.3)
@@
 	)
 	(via
-		(at 77.8 51.6)
+		(at 59.8 46.6)
 		(size 0.6)
 		(drill 0.3)
@@
 	)
 	(via
-		(at 78 57.6)
-		(size 0.6)
-		(drill 0.3)
-		(layers "F.Cu" "B.Cu")
-		(free yes)
-		(net 2)
-	)
-	(via
 		(at 84 36)
 		(size 0.6)
@@
 	)
 	(via
-		(at 79.2 50.4)
-		(size 0.6)
-		(drill 0.3)
-		(layers "F.Cu" "B.Cu")
-		(free yes)
-		(net 2)
-	)
-	(via
 		(at 63 62.8)
 		(size 0.6)
@@
 	)
 	(via
-		(at 77.8 53.6)
-		(size 0.6)
-		(drill 0.3)
-		(layers "F.Cu" "B.Cu")
-		(free yes)
-		(net 2)
-	)
-	(via
 		(at 99 49.6)
 		(size 0.6)
@@
 	)
 	(via
-		(at 81 52.4)
-		(size 0.6)
-		(drill 0.3)
-		(layers "F.Cu" "B.Cu")
-		(free yes)
-		(net 2)
-	)
-	(via
 		(at 66.8 51.2)
 		(size 0.6)
@@
 	)
 	(via
-		(at 77.8 52.6)
-		(size 0.6)
-		(drill 0.3)
-		(layers "F.Cu" "B.Cu")
-		(free yes)
-		(net 2)
-	)
-	(via
 		(at 99 43)
 		(size 0.6)
@@
 	)
 	(via
-		(at 77.8 50.6)
+		(at 73 63.2)
 		(size 0.6)
 		(drill 0.3)
@@
 	)
 	(via
-		(at 73 63.2)
+		(at 75.25 57.75)
 		(size 0.6)
 		(drill 0.3)
@@
 	)
 	(via
-		(at 74.8 57.8)
+		(at 56 60.8)
 		(size 0.6)
 		(drill 0.3)
@@
 	)
 	(via
-		(at 56 60.8)
+		(at 76.75 49.5)
 		(size 0.6)
 		(drill 0.3)
@@
 	)
 	(segment
-		(start 75.975 58.8)
-		(end 78 58.8)
+		(start 77.5 55.925)
+		(end 77.5 58.8)
 		(width 1)
 		(layer "F.Cu")
@@
 	)
 	(segment
-		(start 76 55.8375)
-		(end 76 58.775)
+		(start 77.5 58.8)
+		(end 75.8 58.8)
 		(width 1)
 		(layer "F.Cu")
@@
 	)
 	(segment
-		(start 76 58.775)
-		(end 75.975 58.8)
+		(start 75.8 58.8)
+		(end 75.75 58.75)
 		(width 1)
 		(layer "F.Cu")
@@
 	)
 	(segment
-		(start 78.725 55.925)
-		(end 79.6 55.05)
+		(start 76 54.959204)
+		(end 80.359204 50.6)
 		(width 1)
 		(layer "F.Cu")
@@
 	)
 	(segment
-		(start 77.5 55.925)
-		(end 78.725 55.925)
+		(start 76 55.8375)
+		(end 76 54.959204)
 		(width 1)
 		(layer "F.Cu")
@@
 	)
 	(segment
-		(start 79.6 55.05)
-		(end 79.6 51.8)
+		(start 80.4 57.6)
+		(end 80.4 55.652)
 		(width 1)
 		(layer "F.Cu")
@@
 	)
 	(segment
-		(start 78.725 55.925)
-		(end 80.4 57.6)
+		(start 78.822 54.074)
+		(end 76.885204 54.074)
 		(width 1)
 		(layer "F.Cu")
@@
 	)
 	(segment
-		(start 80.8 50.6)
-		(end 84.4 50.6)
+		(start 80.4 63.3)
+		(end 81.4 64.3)
 		(width 1)
 		(layer "F.Cu")
@@
 	)
 	(segment
-		(start 80.4 63.3)
-		(end 81.4 64.3)
+		(start 76.885204 54.074)
+		(end 76 54.959204)
 		(width 1)
 		(layer "F.Cu")
@@
 	)
 	(segment
-		(start 79.6 51.8)
-		(end 80.8 50.6)
+		(start 80.359204 50.6)
+		(end 84.4 50.6)
 		(width 1)
 		(layer "F.Cu")
@@
 	)
 	(segment
+		(start 80.4 55.652)
+		(end 78.822 54.074)
+		(width 1)
+		(layer "F.Cu")
+		(net 6)
+	)
+	(segment
+		(start 76 53.75)
+		(end 76 55.8375)
+		(width 1)
+		(layer "F.Cu")
+		(net 6)
+	)
+	(segment
 		(start 91.4 66.925)
 		(end 96.63 66.925)
@@
 		(layer "F.Cu")
 		(hatch edge 0.5)
-		(connect_pads yes
+		(connect_pads
 			(clearance 0.5)
 		)
@@
 		(hatch edge 0.5)
 		(priority 1)
-		(connect_pads yes
+		(connect_pads
 			(clearance 0.5)
 		)
